File: pcb/3buttons-3lights-v1.brd (EAGLE design)
At the start: 76.2 x 25.4 mm, 17 parts

Commit message: designing circuit boards
Other:
- board text added: "3buttons-3lights-v1"
- board text removed: "BUTTON INDICATOR BOARD V1"
Changed lines of the file:
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@@
 <wire x1="0" y1="0" x2="76.2" y2="0" width="0" layer="20"/>
 <wire x1="76.2" y1="0" x2="76.2" y2="25.4" width="0" layer="20"/>
-<text x="58.42" y="2.54" size="1.778" layer="21" rot="R180">BUTTON INDICATOR BOARD V1</text>
+<text x="58.42" y="2.54" size="1.778" layer="21" rot="R180">3buttons-3lights-v1</text>
 <text x="75.565" y="20.955" size="1.27" layer="21" rot="R180">GND</text>
 <text x="73.025" y="15.875" size="1.27" layer="21" rot="R180">DIN</text>
